File: hardware/KiCAD/scampi.kicad_sch (KiCad schematic)
At the start: 58 parts, among them IC1 LSF0204GU12X, J1 AudioJack3_SwitchT, U1 MIC5365-1.8YC5-TR, U2 TLV320AIC3100, U3 ATTINY1616-MNR

Commit message: board tweaks & firmware
Parts:
- added C17, C18: 47µF, Capacitor_SMD:C_0603_1608Metric, symbol Device:C_Small
- C13, C14: value 0.47µF -> 1µF
Connections:
- net HPL: now also C17.2; no longer U2.27 (HPL)
- net HPR: now also C18.2; no longer U2.30 (HPR)
- new net: C17.1, U2.27 (HPL)
- new net: C18.1, U2.30 (HPR)
Other:
- moved on the sheet: DET1, HPL1, HPR1, R1, TP8, TP9
