File: KiCAD/scampi.kicad_sch (KiCad schematic)
At the start: 57 parts, among them IC1 LSF0204GU12X, J2 PJ-320D, U1 MIC5365-1.8YC5-TR, U2 TLV320AIC3100, U3 ATTINY1616-MNR

Commit message: firmware, new layout
Parts:
- removed C14, C15: 47µF, Capacitor_SMD:C_0603_1608Metric, symbol Device:C_Small
- removed J2: PJ-320D, SamacSys_Parts:Jack_3.5mm_PJ320D_Horizontal, symbol Connector_Audio:AudioJack4
- added DET1, HPL1, HPR1: ~, SamacSys_Parts:pth_pad, symbol Connector:TestPoint
- added J1: AudioJack3_SwitchT, Connector_Audio:Jack_3.5mm_CUI_SJ-3524-SMT_Horizontal, symbol Connector_Audio:AudioJack3_SwitchT
- C13: renamed from C16; value 1µF -> 0.47µF
- C14: renamed from C17; value 1µF -> 0.47µF
- renumbered C18 to C15, C13 to C16, R2 to R1, R3 to R2, R4 to R3, R1 to R4, TP5 to TP1, TP14 to TP10, TP15 to TP11, TP16 to TP12, TP17 to TP13, TP18 to TP14, TP1 to TP15, TP2 to TP16, TP3 to TP17, TP4 to TP18, TP6 to TP2, TP7 to TP3, TP8 to TP4, TP9 to TP5, TP10 to TP6, TP11 to TP7, TP12 to TP8, TP13 to TP9
Connections:
- net C_IN: now also IC1.3 (A2); no longer IC1.4 (A3)
- net GND: now also J1.S
- net HPL: now also U2.27 (HPL), HPL1.1, J1.T
- net HPR: now also U2.30 (HPR), HPR1.1, J1.R
- net HPS: now also DET1.1, J1.TN
- net W_IN: now also IC1.4 (A3); no longer IC1.3 (A2)
Other:
- moved on the sheet: R1, TP8, TP9
